Commit message: Neue Bahngruppen und Intrinsic-Fahrten hinzugefügt. Dokumentation erweitert. Aufräumarbeiten in der URDF-GUI und in den Tests. README.md hinzugefügt. Neue Dateien

File: bmKinematic.urdf (robot description, URDF)
Before this commit: robot my_robot, 12 links, 11 joints
Links:
- removed link tcp11
- added link link12
Joints:
- removed joint frame10
- added joint TCP_link: type fixed, parent link_11, child link12, origin xyz=0 0.1 0.1 rpy=0 0 0
