Commit message: Installation: Anwenden/Prüfen/Fehlerfall, Projekt vor ROS und Wrapper
- Installationsschritte (2.1 bis 2.6, Anhang B) in Anwenden, Prüfen und
  Fehlerfall gegliedert, mit farbigen Blöcken in der PDF
- Projekt herunterladen jetzt vor ROS/MoveIt und Wrapper (neu 2.3), weil
  Pilz-Patch und Wrapper das Projekt brauchen; Verweise angepasst
- Kontrolle von WSL und VM-Plattform als ein einzeiliger Befehl
- Virtualisierung der CPU prüfen: Task-Manager und systeminfo, Weg ins UEFI
- Kurze Inline-Befehle in der PDF nicht mehr umbrechen (befehle_ganz.lua)
- Überlange Befehlszeile in der README gekürzt
- Neue Bahnen und URDF-Sicherung; Gelenk joint1 in Q1 umbenannt

Co-Authored-By: Claude Opus 5.5 <noreply@anthropic.com>

File: bmKinematic.urdf (robot description, URDF)
Before this commit: robot my_robot, 12 links, 11 joints
Joints:
- removed joint joint1
- added joint Q1: type revolute, parent base_link, child link_1, origin xyz=0 0 0.05 rpy=0 0 0, axis 0 0 1, limit lower=-3.14159 upper=3.14159 effort=10 velocity=1.0
